Commit message: 1.更新urdf碰撞体

File: resources/elf2/urdf/elf2_dof12.urdf (robot description, URDF)
Before this commit: robot elf2, 26 links, 25 joints
Links:
- link l_ankle_y_link: geometry visual mesh filename=../meshes/l_ankle_y_link.STL
- link l_hip_x_link: geometry visual mesh filename=../meshes/l_hip_x_link.STL
- link l_hip_y_link: geometry visual mesh filename=../meshes/l_hip_y_link.STL
- link l_hip_z_link: geometry visual mesh filename=../meshes/l_hip_z_link.STL
- link l_shld_x_link: geometry visual mesh filename=../meshes/l_shld_x_link.STL
- link l_shld_y_link: geometry visual mesh filename=../meshes/l_shld_y_link.STL
- link r_ankle_y_link: geometry visual mesh filename=../meshes/r_ankle_y_link.STL
- link r_hip_x_link: geometry visual mesh filename=../meshes/r_hip_x_link.STL
- link r_hip_y_link: geometry visual mesh filename=../meshes/r_hip_y_link.STL
- link r_hip_z_link: geometry visual mesh filename=../meshes/r_hip_z_link.STL
- link r_shld_x_link: geometry visual mesh filename=../meshes/r_shld_x_link.STL
- link r_shld_y_link: geometry visual mesh filename=../meshes/r_shld_y_link.STL
- link waist_x_link: geometry visual mesh filename=../meshes/waist_x_link.STL
- link waist_z_link: geometry visual mesh filename=../meshes/waist_z_link.STL

File: resources/elf2/urdf/elf2_dof25.urdf (robot description, URDF)
Before this commit: robot elf2, 26 links, 25 joints
Links:
- link l_ankle_y_link: geometry visual mesh filename=../meshes/l_ankle_y_link.STL
- link l_hip_x_link: geometry visual mesh filename=../meshes/l_hip_x_link.STL
- link l_hip_y_link: geometry visual mesh filename=../meshes/l_hip_y_link.STL
- link l_hip_z_link: geometry visual mesh filename=../meshes/l_hip_z_link.STL
- link l_shld_x_link: geometry visual mesh filename=../meshes/l_shld_x_link.STL
- link l_shld_y_link: geometry visual mesh filename=../meshes/l_shld_y_link.STL
- link r_ankle_y_link: geometry visual mesh filename=../meshes/r_ankle_y_link.STL
- link r_hip_x_link: geometry visual mesh filename=../meshes/r_hip_x_link.STL
- link r_hip_y_link: geometry visual mesh filename=../meshes/r_hip_y_link.STL
- link r_hip_z_link: geometry visual mesh filename=../meshes/r_hip_z_link.STL
- link r_shld_x_link: geometry visual mesh filename=../meshes/r_shld_x_link.STL
- link r_shld_y_link: geometry visual mesh filename=../meshes/r_shld_y_link.STL
- link waist_x_link: geometry visual mesh filename=../meshes/waist_x_link.STL
- link waist_z_link: geometry visual mesh filename=../meshes/waist_z_link.STL
