Commit message: 1.update sensor urdf

File: resources/elf2-trunk/urdf/elf2_trunk_dof12.urdf (robot description, URDF)
Before this commit: robot elf2, 26 links, 25 joints
Links:
- added link d435i
- added link mid360
Joints:
- added joint d435i_joint: type fixed, parent base_link, child d435i, origin xyz=0.03255 0 0.2818 rpy=-1.5708 0 -1.5708, axis 0 0 0
- added joint mid360_joint: type fixed, parent base_link, child mid360, origin xyz=0 0 0.23988 rpy=3.1416 0 1.5708, axis 0 0 0

File: resources/elf2-trunk/urdf/elf2_trunk_dof25.urdf (robot description, URDF)
Before this commit: robot elf2, 26 links, 25 joints
Links:
- added link d435i
- added link mid360
Joints:
- added joint d435i_joint: type fixed, parent base_link, child d435i, origin xyz=0.03255 0 0.2818 rpy=-1.5708 0 -1.5708, axis 0 0 0
- added joint mid360_joint: type fixed, parent base_link, child mid360, origin xyz=0 0 0.23988 rpy=3.1416 0 1.5708, axis 0 0 0
